File: mega-wifi.kicad_pcb (KiCad board)
At the start: 2 copper layers, 83.8 x 50.2 mm, 51 parts, among them P1 CONN_01X02, P2 MD-CART-FINGERS, Q1 2N7002, U1 SC16C550BIB48, U2 S29GL032N, U3 ESP-12E, U4 AZ1117CH-3.3, U5 74LVC1G08GW, U6 74LVC162245, U7 74LVC245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

Commit message: Updated to latest KiCad and libraries version.
Changed lines of the file:
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@@
-(kicad_pcb (version 20170123) (host pcbnew "(2017-02-04 revision 9a6e5734b)-master")
+(kicad_pcb (version 20171130) (host pcbnew "(5.0.0-rc2-dev-347-g62c5a706d)")
   (general
-    (links 235)
-    (no_connects 1)
-    (area 104.039999 79.909999 188.060001 130.275001)
     (thickness 1.6)
     (drawings 24)
@@
       (layerselection 0x010e8_ffffffff)
       (usegerberextensions false)
+      (usegerberattributes false)
+      (usegerberadvancedattributes false)
+      (creategerberjobfile false)
       (excludeedgelayer true)
       (linewidth 0.100000)
@@
     (model TO_SOT_Packages_SMD.3dshapes/SOT-223.wrl
       (at (xyz 0 0 0))
-      (scale (xyz 0.4 0.4 0.4))
-      (rotate (xyz 0 0 0))
+      (scale (xyz 1 1 1))
+      (rotate (xyz 0 0 -90))
     )
   )
@@
       (net 46 /WiFi/W_TX))
     (model /home/jalon/src/github/kicad/lib/kicad-ESP8266/ESP8266.3dshapes/ESP-12.wrl
-      (at (xyz 0.047 0 0))
+      (offset (xyz 1.193799982070923 0 0))
       (scale (xyz 0.3937 0.3937 0.3937))
       (rotate (xyz 0 0 0))
@@
       (rotate (xyz 0 0 0))
     )
+    (model ${KISYS3DMOD}/Crystals.3dshapes/Crystal_SMD_HC49-SD-2pin.wrl
+      (at (xyz 0 0 0))
+      (scale (xyz 1 1 1))
+      (rotate (xyz 0 0 0))
+    )
   )
   (module doragasu:HOLE_245 locked (layer F.Cu)
@@
     (pad 2 smd rect (at -1.80086 0) (size 2.60096 1.6002) (layers F.Cu F.Paste F.Mask)
       (net 2 GND))
-    (model Capacitors_SMD.3dshapes/c_elec_4x4.5.wrl
+    (model ${KISYS3DMOD}/Capacitors_SMD.3dshapes/CP_Elec_4x4.5.step
       (at (xyz 0 0 0))
       (scale (xyz 1 1 1))
@@
     (pad 2 smd rect (at -1.80086 0) (size 2.60096 1.6002) (layers F.Cu F.Paste F.Mask)
       (net 2 GND))
-    (model Capacitors_SMD.3dshapes/c_elec_4x4.5.wrl
+    (model ${KISYS3DMOD}/Capacitors_SMD.3dshapes/CP_Elec_4x4.5.step
       (at (xyz 0 0 0))
       (scale (xyz 1 1 1))
@@
       (xy 0.40501 0.04038) (xy 0.57493 -0.11624) (xy 1.68398 -0.11624)) (layer F.Mask) (width 0.01))
     (fp_poly (pts (xy 0.27241 -0.10502) (xy 0.38195 -1.33348) (xy 0.66922 -1.02016) (xy 0.59468 -0.18477)
-      (xy 0.38119 0.01195) (xy 0.27241 -0.10502) (xy 0.27241 -0.10502)) (layer F.Cu) (width 0.01))
+      (xy 0.38119 0.01195) (xy 0.27241 -0.10502)) (layer F.Cu) (width 0.01))
     (fp_poly (pts (xy 0.27241 -0.10502) (xy 0.38195 -1.33348) (xy 0.66922 -1.02016) (xy 0.59468 -0.18477)
-      (xy 0.38119 0.01195) (xy 0.27241 -0.10502) (xy 0.27241 -0.10502)) (layer F.Mask) (width 0.01))
+      (xy 0.38119 0.01195) (xy 0.27241 -0.10502)) (layer F.Mask) (width 0.01))
     (fp_poly (pts (xy 1.82168 1.481847) (xy 0.15583 1.481847) (xy 0.50375 1.168533) (xy 1.53684 1.168533)
       (xy 1.82168 1.481847)) (layer F.Cu) (width 0.01))
@@
       (xy 0.40501 -0.04038) (xy 0.57493 0.11624) (xy 1.68398 0.11624)) (layer B.Mask) (width 0.01))
     (fp_poly (pts (xy 0.27241 0.10502) (xy 0.38195 1.33348) (xy 0.66922 1.02016) (xy 0.59468 0.18477)
-      (xy 0.38119 -0.01195) (xy 0.27241 0.10502) (xy 0.27241 0.10502)) (layer B.Mask) (width 0.01))
+      (xy 0.38119 -0.01195) (xy 0.27241 0.10502)) (layer B.Mask) (width 0.01))
     (fp_poly (pts (xy 1.82168 -1.481847) (xy 0.15583 -1.481847) (xy 0.50375 -1.168533) (xy 1.53684 -1.168533)
       (xy 1.82168 -1.481847)) (layer B.Mask) (width 0.01))
@@
       (net 2 GND))
     (model Socket_Strips/Socket_Strip_Straight_1x02.wrl
-      (at (xyz 0.05 0 0))
+      (offset (xyz 1.269999980926514 0 0))
       (scale (xyz 1 1 1))
       (rotate (xyz 0 0 180))
@@
     (pad 2 smd rect (at 0.81 0 270) (size 1.38 1.25) (layers F.Cu F.Paste F.Mask)
       (net 62 "Net-(P2-PadB3)"))
-    (model Capacitors_SMD/C_0805.wrl
+    (model Resistors_SMD.3dshapes/R_0805.wrl
       (at (xyz 0 0 0))
       (scale (xyz 1 1 1))
@@
     (polygon
       (pts
-        (xy 172.6692 111.7854) (xy 174.5742 111.7854) (xy 174.5742 112.4204) (xy 172.6692 112.4204) (xy 172.6692 112.4204)
+        (xy 172.6692 111.7854) (xy 174.5742 111.7854) (xy 174.5742 112.4204) (xy 172.6692 112.4204)
       )
     )
