File: mega-wifi.kicad_pcb (KiCad board)
At the start: 2 copper layers, 83.8 x 50.2 mm, 51 parts, among them P1 CONN_01X02, P2 MD-CART-FINGERS, Q1 2N7002, U1 SC16C550BIB48, U2 S29GL032N, U3 ESP-12E, U4 AZ1117CH-3.3, U5 74LVC1G08GW, U6 74LVC162245, U7 74LVC245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

Commit message: Update to Rev.A2
Parts:
- C3, C4: value NP -> 22p
- C5: value 100n -> NP
- D1: value LED -> NP
- P1: value CONN_01X02 -> NP; footprint Socket_Strips:Socket_Strip_Straight_1x02 -> Connector_PinHeader_2.54mm:PinHeader_1x02_P2.54mm_Vertical
- R10, R9: value 10k -> NP
- R12, R13: value 47k -> NP
- R14, R16, R18: value 0 -> NP
- R4: value 1k -> NP
- R8: value 220 -> NP
- Y1: value NP -> 24 MHz
- turned P1 to 180 degrees
Connections:
- P2 pad B10: Net-(P2-PadB10) -> (no net)
- P2 pad B11: Net-(P2-PadB11) -> (no net)
- P2 pad B12: Net-(P2-PadB12) -> (no net)
- P2 pad B15: Net-(P2-PadB15) -> (no net)
- P2 pad B2: Net-(P2-PadB2) -> (no net)
- P2 pad B20: Net-(P2-PadB20) -> (no net)
- P2 pad B21: Net-(P2-PadB21) -> (no net)
- P2 pad B26: Net-(P2-PadB26) -> (no net)
- P2 pad B29: Net-(P2-PadB29) -> (no net)
- P2 pad B30: Net-(P2-PadB30) -> (no net)
- U1 pad 1: Net-(U1-Pad1) -> (no net)
- U1 pad 13: Net-(U1-Pad13) -> (no net)
- U1 pad 21: Net-(U1-Pad21) -> (no net)
- U1 pad 22: Net-(U1-Pad22) -> (no net)
- U1 pad 23: Net-(U1-Pad23) -> (no net)
- U1 pad 25: Net-(U1-Pad25) -> (no net)
- U1 pad 29: Net-(U1-Pad29) -> (no net)
- U1 pad 30: Net-(U1-Pad30) -> (no net)
- U1 pad 36: Net-(U1-Pad36) -> (no net)
- U1 pad 37: Net-(U1-Pad37) -> (no net)
- U1 pad 40: Net-(U1-Pad40) -> (no net)
- U1 pad 41: Net-(U1-Pad41) -> (no net)
- U1 pad 48: Net-(U1-Pad48) -> (no net)
- U1 pad 6: Net-(U1-Pad6) -> (no net)
- U2 pad 13: Net-(U2-Pad13) -> (no net)
- U2 pad 14: Net-(U2-Pad14) -> (no net)
- U2 pad 15: Net-(U2-Pad15) -> (no net)
- U3 pad 10: Net-(U3-Pad10) -> (no net)
- U3 pad 11: Net-(U3-Pad11) -> (no net)
- U3 pad 12: Net-(U3-Pad12) -> (no net)
- U3 pad 13: Net-(U3-Pad13) -> (no net)
- U3 pad 14: Net-(U3-Pad14) -> (no net)
- U3 pad 2: Net-(U3-Pad2) -> (no net)
- U3 pad 9: Net-(U3-Pad9) -> (no net)
Other:
- board size 83.8 x 50.2 mm -> 83.8 x 51 mm
- board text added: "MeGaWiFi Rev.A2 (2021)"
- board text added: "doragasu (2021)"
- board text removed: "License: CERN OHL 1.2"
- board text removed: "MeGaWiFi Rev.A1 (2016)"
- board text removed: "doragasu (2016)"
