File: mega-wifi.sch (KiCad schematic (older format))
At the start: 25 parts, among them P2 MD-CART-FINGERS, U4 AZ1117CH-3.3, U5 74LVC1G08GW, U6 74LVC162245, U7 74LVC245, U8 74LVC162245

Commit message: Updated to latest KiCad and libraries version.
Parts:
- C10, C11, C12, C13, C15, C8, C9: symbol C -> device:C
- C14, C7: symbol CP -> device:CP
- P2: symbol MD-CART-FINGERS -> doragasu:MD-CART-FINGERS
- R10, R11, R12, R13, R14, R15, R16, R17, R18, R9: symbol R -> device:R
- U4: symbol AZ1117CH -> doragasu:AZ1117CH
- U5: symbol 74LVC1G08GW -> doragasu:74LVC1G08GW
- U6, U8: symbol 74LVC162245 -> doragasu:74LVC162245
- U7: symbol 74LVC245 -> doragasu:74LVC245
Changed lines of the file:
@@
-EESchema Schematic File Version 2
-LIBS:power
-LIBS:device
-LIBS:transistors
-LIBS:conn
-LIBS:linear
-LIBS:regul
-LIBS:74xx
-LIBS:cmos4000
-LIBS:adc-dac
-LIBS:memory
-LIBS:xilinx
-LIBS:microcontrollers
-LIBS:dsp
-LIBS:microchip
-LIBS:analog_switches
-LIBS:motorola
-LIBS:texas
-LIBS:intel
-LIBS:audio
-LIBS:interface
-LIBS:digital-audio
-LIBS:philips
-LIBS:display
-LIBS:cypress
-LIBS:siliconi
-LIBS:opto
-LIBS:atmel
-LIBS:contrib
-LIBS:valves
-LIBS:ESP8266
-LIBS:doragasu
+EESchema Schematic File Version 4
 LIBS:mega-wifi-cache
 EELAYER 26 0
@@
 $EndDescr
 $Comp
-L MD-CART-FINGERS P2
+L doragasu:MD-CART-FINGERS P2
 U 1 1 56179054
 P 2450 4850
@@
 $EndComp
 $Comp
-L 74LVC162245 U6
+L doragasu:74LVC162245 U6
 U 2 1 561938BA
 P 4750 3150
@@
 $EndComp
 $Comp
-L 74LVC162245 U6
+L doragasu:74LVC162245 U6
 U 1 1 5619397A
 P 4750 1750
@@
 $EndComp
 $Comp
-L 74LVC162245 U8
+L doragasu:74LVC162245 U8
 U 2 1 56193A0C
 P 4750 7350
@@
 	3750 5050 3850 4950
 $Comp
-L 74LVC162245 U8
+L doragasu:74LVC162245 U8
 U 1 1 56196C4D
 P 4750 5950
@@
 C_CLK
 $Comp
-L C C8
+L device:C C8
 U 1 1 561DA569
 P 1400 2900
@@
 $EndComp
 $Comp
-L CP C7
+L device:CP C7
 U 1 1 561DA6C6
 P 1150 2900
@@
 $EndComp
 $Comp
-L GND #PWR4
+L power:GND #PWR4
 U 1 1 561DDDFF
 P 1400 3200
@@
 $EndComp
 $Comp
-L +5V #PWR2
+L power:+5V #PWR2
 U 1 1 561DF187
 P 1400 2600
@@
 $EndComp
 $Comp
-L GND #PWR1
+L power:GND #PWR1
 U 1 1 561E4A8B
 P 5450 1350
@@
 $EndComp
 $Comp
-L GND #PWR3
+L power:GND #PWR3
 U 1 1 561E5F8F
 P 5450 2750
@@
 $EndComp
 $Comp
-L GND #PWR5
+L power:GND #PWR5
 U 1 1 561E6B00
 P 5450 4150
@@
 #W
 $Comp
-L R R11
+L device:R R11
 U 1 1 5620771C
 P 1350 5400
@@
 $EndComp
 $Comp
-L R R15
+L device:R R15
 U 1 1 56207A0F
 P 1500 5150
@@
 $EndComp
 $Comp
-L GND #PWR6
+L power:GND #PWR6
 U 1 1 56212D5A
 P 1350 5550
@@
 3.3V linear regulator,\nIlimit,min = 1 A
 $Comp
-L C C9
+L device:C C9
 U 1 1 5625E0C9
 P 1700 9700
@@
 $EndComp
 $Comp
-L C C10
+L device:C C10
 U 1 1 5625E8FF
 P 2000 9700
@@
 $EndComp
 $Comp
-L C C11
+L device:C C11
 U 1 1 5625EA93
 P 2300 9700
@@
 $EndComp
 $Comp
-L C C12
+L device:C C12
 U 1 1 5625EC22
 P 2600 9700
@@
 $EndComp
 $Comp
-L C C13
+L device:C C13
 U 1 1 5625EDB4
 P 2900 9700
@@
 $EndComp
 $Comp
-L GND #PWR10
+L power:GND #PWR10
 U 1 1 562608DD
 P 2450 10000
@@
 $EndComp
 $Comp
-L VCC #PWR9
+L power:VCC #PWR9
 U 1 1 56262FCA
 P 2450 9400
@@
 $EndComp
 $Comp
-L R R14
+L device:R R14
 U 1 1 561B880E
 P 1500 4750
@@
 	1050 8650 6150 8650
 Wire Wire Line
-	1650 3050 1650 3550
+	1650 3050 1650 3150
 Connection ~ 1650 3250
 Connection ~ 1650 3150
@@
 	1650 2650 1650 2750
 Wire Wire Line
-	1150 2650 1650 2650
+	1150 2650 1400 2650
 Wire Wire Line
 	1150 2650 1150 2750
@@
 	1150 3050 1150 3150
 Wire Wire Line
-	1150 3150 1650 3150
-Wire Wire Line
-	1400 3050 1400 3200
+	1150 3150 1400 3150
+Wire Wire Line
+	1400 3050 1400 3150
 Connection ~ 1400 3150
 Wire Wire Line
-	1400 2600 1400 2750
+	1400 2600 1400 2650
 Connection ~ 1400 2650
 Connection ~ 1650 2650
@@
 Wire Wire Line
 	1250 8550 5850 8550
-Wire Bus Line
-	3750 1650 3750 8150
 Wire Wire Line
 	1350 5150 1350 5250
@@
 	1700 9550 1700 9450
 Wire Wire Line
-	1700 9450 3200 9450
+	1700 9450 2000 9450
 Wire Wire Line
 	2900 9450 2900 9550
@@
 	1700 9850 1700 9950
 Wire Wire Line
-	1700 9950 3200 9950
+	1700 9950 2000 9950
 Wire Wire Line
 	2900 9950 2900 9850
@@
 UART mapped at 0xA130C1 (#C_TIME range).
 $Comp
-L AZ1117CH U4
+L doragasu:AZ1117CH U4
 U 1 1 56203BD5
 P 1150 10700
@@
 Locate caps near the 3.3V regulator input.\n
 $Comp
-L +5V #PWR11
+L power:+5V #PWR11
 U 1 1 56207F25
 P 700 10600
@@
 	700  10650 750  10650
 $Comp
-L GND #PWR13
+L power:GND #PWR13
 U 1 1 56209B97
 P 1150 11050
@@
 $EndComp
 $Comp
-L CP C14
+L device:CP C14
 U 1 1 5620A5AC
 P 1800 10800
@@
 Connection ~ 1150 10950
 $Comp
-L VCC #PWR12
+L power:VCC #PWR12
 U 1 1 5620D239
 P 1800 10600
@@
 A19
 NoConn ~ 1650 4850
-Wire Bus Line
-	5650 1650 5650 8450
 Wire Wire Line
 	5750 8350 6150 8350
@@
 #OE
 $Comp
-L C C15
+L device:C C15
 U 1 1 5695B5C9
 P 3200 9700
@@
 	5650 8450 5750 8350
 Wire Wire Line
-	3250 7650 3650 7650
+	3250 7650 3550 7650
 Wire Wire Line
 	3250 7450 3650 7450
@@
 	3650 7650 3750 7750
 Wire Wire Line
-	2050 7550 2050 8050
+	2050 7550 2050 7900
 Wire Wire Line
 	2050 8050 3650 8050
@@
 If assembling ONLY Flash (without\nUART), mount R17 instead of U5.
 $Comp
-L 74LVC245 U7
+L doragasu:74LVC245 U7
 U 1 1 562586F6
 P 4750 4550
@@
 #C_TIME
 $Comp
-L 74LVC1G08GW U5
+L doragasu:74LVC1G08GW U5
 U 1 1 569F14E7
 P 2650 7550
@@
 $EndComp
 $Comp
-L R R17
+L device:R R17
 U 1 1 56965CA2
 P 2700 7900
@@
 Connection ~ 3550 7650
 $Comp
-L R R16
+L device:R R16
 U 1 1 56C15D44
 P 1500 6550
@@
 	1650 6550 1650 6650
 Wire Wire Line
-	1350 6550 1350 8750
+	1350 6550 1350 6850
 Wire Wire Line
 	1350 8750 6150 8750
@@
 	950  4450 950  8850
 Wire Wire Line
-	950  8850 6150 8850
-Wire Wire Line
-	850  4150 850  9000
+	950  8850 1100 8850
+Wire Wire Line
+	850  4150 850  8950
 Wire Wire Line
 	850  8950 6150 8950
 $Comp
-L R R12
+L device:R R12
 U 1 1 56C2EF02
 P 1500 4150
@@
 $EndComp
 $Comp
-L R R13
+L device:R R13
 U 1 1 56C2F106
 P 1500 4450
@@
 	1350 4450 950  4450
 $Comp
-L R R9
+L device:R R9
 U 1 1 56C318B7
 P 850 9150
@@
 $EndComp
 $Comp
-L R R10
+L device:R R10
 U 1 1 56C344D0
 P 1100 9150
@@
 Connection ~ 1100 8850
 $Comp
-L GND #PWR8
+L power:GND #PWR8
 U 1 1 56C372F3
 P 1100 9300
@@
 $EndComp
 $Comp
-L GND #PWR7
+L power:GND #PWR7
 U 1 1 56C37650
 P 850 9300
@@
 	1    0    0    -1
 $EndComp
-Wire Wire Line
-	850  9300 850  9300
-Wire Wire Line
-	1100 9300 1100 9300
 $Sheet
 S 6150 6350 1000 2700
@@
 NoConn ~ 3250 6950
 $Comp
-L R R18
+L device:R R18
 U 1 1 57A27ECE
 P 1500 6850
@@
 $EndComp
 Connection ~ 1350 6850
+Wire Wire Line
+	1650 3250 1650 3550
+Wire Wire Line
+	1650 3150 1650 3250
+Wire Wire Line
+	1400 3150 1650 3150
+Wire Wire Line
+	1400 3150 1400 3200
+Wire Wire Line
+	1400 2650 1650 2650
+Wire Wire Line
+	1400 2650 1400 2750
+Wire Wire Line
+	2600 9450 2900 9450
+Wire Wire Line
+	2300 9450 2450 9450
+Wire Wire Line
+	2000 9450 2300 9450
+Wire Wire Line
+	2000 9950 2300 9950
+Wire Wire Line
+	2300 9950 2450 9950
+Wire Wire Line
+	2600 9950 2900 9950
+Wire Wire Line
+	2900 9450 3200 9450
+Wire Wire Line
+	2900 9950 3200 9950
+Wire Wire Line
+	2450 9450 2600 9450
+Wire Wire Line
+	2450 9950 2600 9950
+Wire Wire Line
+	2050 7900 2050 8050
+Wire Wire Line
+	3550 7650 3650 7650
+Wire Wire Line
+	850  8950 850  9000
+Wire Wire Line
+	1100 8850 6150 8850
+Wire Wire Line
+	1350 6850 1350 8750
+Wire Bus Line
+	3750 1650 3750 8150
+Wire Bus Line
+	5650 1650 5650 8450
 $EndSCHEMATC

Commit message: Update schematic components to latest library
Parts:
- C10, C11, C12, C13, C15, C8, C9: symbol device:C -> Device:C
- C14, C7: symbol device:CP -> Device:CP
- R10, R11, R12, R13, R14, R15, R16, R17, R18, R9: symbol device:R -> Device:R
Changed lines of the file:
@@
 EESchema Schematic File Version 4
-LIBS:mega-wifi-cache
-EELAYER 26 0
+EELAYER 30 0
 EELAYER END
 $Descr A4 8268 11693 portrait
@@
 C_CLK
 $Comp
-L device:C C8
+L Device:C C8
 U 1 1 561DA569
 P 1400 2900
@@
 $EndComp
 $Comp
-L device:CP C7
+L Device:CP C7
 U 1 1 561DA6C6
 P 1150 2900
@@
 #W
 $Comp
-L device:R R11
+L Device:R R11
 U 1 1 5620771C
 P 1350 5400
@@
 $EndComp
 $Comp
-L device:R R15
+L Device:R R15
 U 1 1 56207A0F
 P 1500 5150
@@
 3.3V linear regulator,\nIlimit,min = 1 A
 $Comp
-L device:C C9
+L Device:C C9
 U 1 1 5625E0C9
 P 1700 9700
@@
 $EndComp
 $Comp
-L device:C C10
+L Device:C C10
 U 1 1 5625E8FF
 P 2000 9700
@@
 $EndComp
 $Comp
-L device:C C11
+L Device:C C11
 U 1 1 5625EA93
 P 2300 9700
@@
 $EndComp
 $Comp
-L device:C C12
+L Device:C C12
 U 1 1 5625EC22
 P 2600 9700
@@
 $EndComp
 $Comp
-L device:C C13
+L Device:C C13
 U 1 1 5625EDB4
 P 2900 9700
@@
 $EndComp
 $Comp
-L device:R R14
+L Device:R R14
 U 1 1 561B880E
 P 1500 4750
@@
 $EndComp
 $Comp
-L device:CP C14
+L Device:CP C14
 U 1 1 5620A5AC
 P 1800 10800
@@
 #OE
 $Comp
-L device:C C15
+L Device:C C15
 U 1 1 5695B5C9
 P 3200 9700
@@
 $EndComp
 $Comp
-L device:R R17
+L Device:R R17
 U 1 1 56965CA2
 P 2700 7900
@@
 Connection ~ 3550 7650
 $Comp
-L device:R R16
+L Device:R R16
 U 1 1 56C15D44
 P 1500 6550
@@
 	850  8950 6150 8950
 $Comp
-L device:R R12
+L Device:R R12
 U 1 1 56C2EF02
 P 1500 4150
@@
 $EndComp
 $Comp
-L device:R R13
+L Device:R R13
 U 1 1 56C2F106
 P 1500 4450
@@
 	1350 4450 950  4450
 $Comp
-L device:R R9
+L Device:R R9
 U 1 1 56C318B7
 P 850 9150
@@
 $EndComp
 $Comp
-L device:R R10
+L Device:R R10
 U 1 1 56C344D0
 P 1100 9150
@@
 NoConn ~ 3250 6950
 $Comp
-L device:R R18
+L Device:R R18
 U 1 1 57A27ECE
 P 1500 6850

Commit message: Update to Rev.A2
Parts:
- C10, C11, C12, C13, C15, C8, C9: LCSC# (none) -> C2830722
- C14, C7: LCSC# (none) -> C250865
- R10, R9: value 10k -> NP
- R11: LCSC# (none) -> C237121
- R12, R13: value 47k -> NP
- R14, R16, R18: value 0 -> NP
- R15: LCSC# (none) -> C144558
- U4: LCSC# (none) -> C351784
- U5: LCSC# (none) -> C434068
- U6, U8: LCSC# (none) -> C6069
- U7: LCSC# (none) -> C393617
Changed lines of the file:
@@
 Sheet 1 3
 Title "MegaWiFi"
-Date "2017-03-24"
-Rev "A1"
+Date "2021-10-31"
+Rev "A2"
 Comp "doragasu"
 Comment1 "License: CERN OHL 1.2"
@@
 F 3 "" H 4750 3150 60  0000 C CNN
 F 4 "74LVC162245ADGG:11" H 4750 3150 60  0001 C CNN "manf#"
+F 5 "C6069" H 4750 3150 50  0001 C CNN "LCSC#"
 	2    4750 3150
 	-1   0    0    1
@@
 F 3 "" H 4750 1750 60  0000 C CNN
 F 4 "74LVC162245ADGG:11" H 4750 1750 60  0001 C CNN "manf#"
+F 5 "C6069" H 4750 1750 50  0001 C CNN "LCSC#"
 	1    4750 1750
 	-1   0    0    1
@@
 F 3 "" H 4750 7350 60  0000 C CNN
 F 4 "74LVC162245ADGG:11" H 4750 7350 60  0001 C CNN "manf#"
+F 5 "C6069" H 4750 7350 50  0001 C CNN "LCSC#"
 	2    4750 7350
 	1    0    0    -1
@@
 F 3 "" H 4750 5950 60  0000 C CNN
 F 4 "74LVC162245ADGG:11" H 4750 5950 60  0001 C CNN "manf#"
+F 5 "C6069" H 4750 5950 50  0001 C CNN "LCSC#"
 	1    4750 5950
 	1    0    0    -1
@@
 F 2 "Capacitors_SMD:C_0805" H 1438 2750 30  0001 C CNN
 F 3 "" H 1400 2900 60  0000 C CNN
+F 4 "C2830722" H 1400 2900 50  0001 C CNN "LCSC#"
 	1    1400 2900
 	1    0    0    -1
@@
 F 4 "493-9779-1-ND" H 1150 2900 60  0001 C CNN "REF_DIGIKEY"
 F 5 "UWJ0J220MCL1GB" H 1150 2900 60  0001 C CNN "manf#"
+F 6 "C250865" H 1150 2900 50  0001 C CNN "LCSC#"
 	1    1150 2900
 	1    0    0    -1
 $EndComp
 $Comp
-L power:GND #PWR4
+L power:GND #PWR04
 U 1 1 561DDDFF
 P 1400 3200
-F 0 "#PWR4" H 1400 2950 50  0001 C CNN
+F 0 "#PWR04" H 1400 2950 50  0001 C CNN
 F 1 "GND" H 1400 3050 50  0001 C CNN
 F 2 "" H 1400 3200 60  0000 C CNN
@@
 $EndComp
 $Comp
-L power:+5V #PWR2
+L power:+5V #PWR02
 U 1 1 561DF187
 P 1400 2600
-F 0 "#PWR2" H 1400 2450 50  0001 C CNN
+F 0 "#PWR02" H 1400 2450 50  0001 C CNN
 F 1 "+5V" H 1400 2740 50  0000 C CNN
 F 2 "" H 1400 2600 60  0000 C CNN
@@
 $EndComp
 $Comp
-L power:GND #PWR1
+L power:GND #PWR01
 U 1 1 561E4A8B
 P 5450 1350
-F 0 "#PWR1" H 5450 1100 50  0001 C CNN
+F 0 "#PWR01" H 5450 1100 50  0001 C CNN
 F 1 "GND" H 5450 1200 50  0001 C CNN
 F 2 "" H 5450 1350 60  0000 C CNN
@@
 $EndComp
 $Comp
-L power:GND #PWR3
+L power:GND #PWR03
 U 1 1 561E5F8F
 P 5450 2750
-F 0 "#PWR3" H 5450 2500 50  0001 C CNN
+F 0 "#PWR03" H 5450 2500 50  0001 C CNN
 F 1 "GND" H 5450 2600 50  0001 C CNN
 F 2 "" H 5450 2750 60  0000 C CNN
@@
 $EndComp
 $Comp
-L power:GND #PWR5
+L power:GND #PWR05
 U 1 1 561E6B00
 P 5450 4150
-F 0 "#PWR5" H 5450 3900 50  0001 C CNN
+F 0 "#PWR05" H 5450 3900 50  0001 C CNN
 F 1 "GND" H 5450 4000 50  0001 C CNN
 F 2 "" H 5450 4150 60  0000 C CNN
@@
 F 3 "" H 1350 5400 30  0000 C CNN
 F 4 "RMCF0805JT100K" H 1350 5400 60  0001 C CNN "manf#"
+F 5 "C237121" H 1350 5400 50  0001 C CNN "LCSC#"
 	1    1350 5400
 	-1   0    0    1
@@
 F 3 "" H 1500 5150 30  0000 C CNN
 F 4 "RMCF0805JT47K0" V 1500 5150 60  0001 C CNN "manf#"
+F 5 "C144558" V 1500 5150 50  0001 C CNN "LCSC#"
 	1    1500 5150
 	0    -1   -1   0
 $EndComp
 $Comp
-L power:GND #PWR6
+L power:GND #PWR06
 U 1 1 56212D5A
 P 1350 5550
-F 0 "#PWR6" H 1350 5300 50  0001 C CNN
+F 0 "#PWR06" H 1350 5300 50  0001 C CNN
 F 1 "GND" H 1350 5400 50  0001 C CNN
 F 2 "" H 1350 5550 60  0000 C CNN
@@
 F 3 "" H 1700 9700 60  0000 C CNN
 F 4 "CL21F104ZBCNNNC" H 1700 9700 60  0001 C CNN "manf#"
+F 5 "C2830722" H 1700 9700 50  0001 C CNN "LCSC#"
 	1    1700 9700
 	1    0    0    -1
@@
 F 2 "Capacitors_SMD:C_0805" H 2038 9550 30  0001 C CNN
 F 3 "" H 2000 9700 60  0000 C CNN
+F 4 "C2830722" H 2000 9700 50  0001 C CNN "LCSC#"
 	1    2000 9700
 	1    0    0    -1
@@
 F 2 "Capacitors_SMD:C_0805" H 2338 9550 30  0001 C CNN
 F 3 "" H 2300 9700 60  0000 C CNN
+F 4 "C2830722" H 2300 9700 50  0001 C CNN "LCSC#"
 	1    2300 9700
 	1    0    0    -1
@@
 F 2 "Capacitors_SMD:C_0805" H 2638 9550 30  0001 C CNN
 F 3 "" H 2600 9700 60  0000 C CNN
+F 4 "C2830722" H 2600 9700 50  0001 C CNN "LCSC#"
 	1    2600 9700
 	1    0    0    -1
@@
 F 2 "Capacitors_SMD:C_0805" H 2938 9550 30  0001 C CNN
 F 3 "" H 2900 9700 60  0000 C CNN
+F 4 "C2830722" H 2900 9700 50  0001 C CNN "LCSC#"
 	1    2900 9700
 	1    0    0    -1
 $EndComp
 $Comp
-L power:GND #PWR10
+L power:GND #PWR010
 U 1 1 562608DD
 P 2450 10000
-F 0 "#PWR10" H 2450 9750 50  0001 C CNN
+F 0 "#PWR010" H 2450 9750 50  0001 C CNN
 F 1 "GND" H 2450 9850 50  0001 C CNN
 F 2 "" H 2450 10000 60  0000 C CNN
@@
 $EndComp
 $Comp
-L power:VCC #PWR9
+L power:VCC #PWR09
 U 1 1 56262FCA
 P 2450 9400
-F 0 "#PWR9" H 2450 9250 50  0001 C CNN
+F 0 "#PWR09" H 2450 9250 50  0001 C CNN
 F 1 "VCC" H 2450 9550 50  0000 C CNN
 F 2 "" H 2450 9400 60  0000 C CNN
@@
 P 1500 4750
 F 0 "R14" V 1400 4750 50  0000 C CNN
-F 1 "0" V 1500 4750 50  0000 C CNN
+F 1 "NP" V 1500 4750 50  0000 C CNN
 F 2 "doragasu:JUMPER_0805" V 1430 4750 30  0001 C CNN
 F 3 "" H 1500 4750 30  0000 C CNN
+F 4 "" H 1500 4750 50  0001 C CNN "LCSC#"
 	1    1500 4750
 	0    1    1    0
@@
 F 4 "AZ1117CH-3.3TRG1DICT-ND" H 1150 10700 60  0001 C CNN "REF_DIGIKEY"
 F 5 "AP2114H-3.3TRG1" H 1150 10700 60  0001 C CNN "manf#"
+F 6 "C351784" H 1150 10700 50  0001 C CNN "LCSC#"
 	1    1150 10700
 	1    0    0    -1
@@
 Locate caps near the 3.3V regulator input.\n
 $Comp
-L power:+5V #PWR11
+L power:+5V #PWR011
 U 1 1 56207F25
 P 700 10600
-F 0 "#PWR11" H 700 10450 50  0001 C CNN
+F 0 "#PWR011" H 700 10450 50  0001 C CNN
 F 1 "+5V" H 700 10740 50  0000 C CNN
 F 2 "" H 700 10600 60  0000 C CNN
@@
 	700  10650 750  10650
 $Comp
-L power:GND #PWR13
+L power:GND #PWR013
 U 1 1 56209B97
 P 1150 11050
-F 0 "#PWR13" H 1150 10800 50  0001 C CNN
+F 0 "#PWR013" H 1150 10800 50  0001 C CNN
 F 1 "GND" H 1150 10900 50  0001 C CNN
 F 2 "" H 1150 11050 60  0000 C CNN
@@
 F 4 "493-9779-1-ND" H 1800 10800 60  0001 C CNN "REF_DIGIKEY"
 F 5 "UWJ0J220MCL1GB" H 1800 10800 60  0001 C CNN "manf#"
+F 6 "C250865" H 1800 10800 50  0001 C CNN "LCSC#"
 	1    1800 10800
 	1    0    0    -1
@@
 Connection ~ 1150 10950
 $Comp
-L power:VCC #PWR12
+L power:VCC #PWR012
 U 1 1 5620D239
 P 1800 10600
-F 0 "#PWR12" H 1800 10450 50  0001 C CNN
+F 0 "#PWR012" H 1800 10450 50  0001 C CNN
 F 1 "VCC" H 1800 10750 50  0000 C CNN
 F 2 "" H 1800 10600 60  0000 C CNN
@@
 F 2 "Capacitors_SMD:C_0805" H 3238 9550 30  0001 C CNN
 F 3 "" H 3200 9700 60  0000 C CNN
+F 4 "C2830722" H 3200 9700 50  0001 C CNN "LCSC#"
 	1    3200 9700
 	1    0    0    -1
@@
 F 4 "568-1584-5-ND" H 4750 4550 60  0001 C CNN "REF_DIGIKEY"
 F 5 "74LVC245APW,112" H 4750 4550 60  0001 C CNN "manf#"
+F 6 " C393617" H 4750 4550 50  0001 C CNN "LCSC#"
 	1    4750 4550
 	-1   0    0    1
@@
 F 3 "" H 2650 7550 60  0000 C CNN
 F 4 "74LVC1G08W5-7" H 2650 7550 60  0001 C CNN "manf#"
+F 5 "C434068" H 2650 7550 50  0001 C CNN "LCSC#"
 	1    2650 7550
 	-1   0    0    1
@@
 P 1500 6550
 F 0 "R16" V 1600 6600 50  0000 R CNN
-F 1 "0" V 1500 6550 50  0000 R CNN
+F 1 "NP" V 1500 6550 50  0000 C CNN
 F 2 "doragasu:JUMPER_0805" V 1430 6550 30  0001 C CNN
 F 3 "" H 1500 6550 30  0000 C CNN
+F 4 "" H 1500 6550 50  0001 C CNN "LCSC#"
 	1    1500 6550
 	0    -1   -1   0
@@
 P 1500 4150
 F 0 "R12" V 1600 4150 50  0000 C CNN
-F 1 "47k" V 1500 4150 50  0000 C CNN
+F 1 "NP" V 1500 4150 50  0000 C CNN
 F 2 "Resistors_SMD:R_0805" V 1430 4150 30  0001 C CNN
 F 3 "" H 1500 4150 30  0000 C CNN
+F 4 "" H 1500 4150 50  0001 C CNN "LCSC#"
 	1    1500 4150
 	0    -1   -1   0
@@
 P 1500 4450
 F 0 "R13" V 1600 4450 50  0000 C CNN
-F 1 "47k" V 1500 4450 50  0000 C CNN
+F 1 "NP" V 1500 4450 50  0000 C CNN
 F 2 "Resistors_SMD:R_0805" V 1430 4450 30  0001 C CNN
 F 3 "" H 1500 4450 30  0000 C CNN
+F 4 "" H 1500 4450 50  0001 C CNN "LCSC#"
 	1    1500 4450
 	0    -1   -1   0
@@
 P 850 9150
 F 0 "R9" H 780 9104 50  0000 R CNN
-F 1 "10k" V 850 9200 50  0000 R CNN
+F 1 "NP" V 850 9200 50  0000 R CNN
 F 2 "Resistors_SMD:R_0805" V 780 9150 30  0001 C CNN
 F 3 "" H 850 9150 30  0000 C CNN
 F 4 "RMCF0805JT10K0" H 850 9150 60  0001 C CNN "manf#"
+F 5 "" H 850 9150 50  0001 C CNN "LCSC#"
 	1    850  9150
 	-1   0    0    1
@@
 P 1100 9150
 F 0 "R10" H 1030 9104 50  0000 R CNN
-F 1 "10k" V 1100 9200 50  0000 R CNN
+F 1 "NP" V 1100 9200 50  0000 R CNN
 F 2 "Resistors_SMD:R_0805" V 1030 9150 30  0001 C CNN
 F 3 "" H 1100 9150 30  0000 C CNN
+F 4 "" H 1100 9150 50  0001 C CNN "LCSC#"
 	1    1100 9150
 	-1   0    0    1
@@
 Connection ~ 1100 8850
 $Comp
-L power:GND #PWR8
+L power:GND #PWR08
 U 1 1 56C372F3
 P 1100 9300
-F 0 "#PWR8" H 1100 9050 50  0001 C CNN
+F 0 "#PWR08" H 1100 9050 50  0001 C CNN
 F 1 "GND" H 1100 9150 50  0001 C CNN
 F 2 "" H 1100 9300 60  0000 C CNN
@@
 $EndComp
 $Comp
-L power:GND #PWR7
+L power:GND #PWR07
 U 1 1 56C37650
 P 850 9300
-F 0 "#PWR7" H 850 9050 50  0001 C CNN
+F 0 "#PWR07" H 850 9050 50  0001 C CNN
 F 1 "GND" H 850 9150 50  0001 C CNN
 F 2 "" H 850 9300 60  0000 C CNN
@@
 P 1500 6850
 F 0 "R18" V 1600 6900 50  0000 R CNN
-F 1 "0" V 1500 6850 50  0000 R CNN
+F 1 "NP" V 1500 6850 50  0000 C CNN
 F 2 "doragasu:JUMPER_0805" V 1430 6850 30  0001 C CNN
 F 3 "" H 1500 6850 30  0000 C CNN
+F 4 "" H 1500 6850 50  0001 C CNN "LCSC#"
 	1    1500 6850
 	0    -1   -1   0
