File: rom.sch (KiCad schematic (older format))
At the start: 2 parts, among them U2 S29GL032N

Commit message: Updated to latest KiCad and libraries version.
Parts:
- C2: symbol C -> device:C
- U2: symbol S29GL032N -> doragasu:S29GL032N
Changed lines of the file:
@@
-EESchema Schematic File Version 2
-LIBS:power
-LIBS:device
-LIBS:transistors
-LIBS:conn
-LIBS:linear
-LIBS:regul
-LIBS:74xx
-LIBS:cmos4000
-LIBS:adc-dac
-LIBS:memory
-LIBS:xilinx
-LIBS:microcontrollers
-LIBS:dsp
-LIBS:microchip
-LIBS:analog_switches
-LIBS:motorola
-LIBS:texas
-LIBS:intel
-LIBS:audio
-LIBS:interface
-LIBS:digital-audio
-LIBS:philips
-LIBS:display
-LIBS:cypress
-LIBS:siliconi
-LIBS:opto
-LIBS:atmel
-LIBS:contrib
-LIBS:valves
-LIBS:ESP8266
-LIBS:doragasu
+EESchema Schematic File Version 4
 LIBS:mega-wifi-cache
 EELAYER 26 0
@@
 $EndDescr
 $Comp
-L S29GL032N U2
+L doragasu:S29GL032N U2
 U 1 1 561A024F
 P 6000 2850
@@
 NoConn ~ 6700 3650
 $Comp
-L VCC #PWR14
+L power:VCC #PWR14
 U 1 1 561C7245
 P 6750 4050
@@
 	6700 4050 6750 4050
 $Comp
-L C C2
+L device:C C2
 U 1 1 561C7483
 P 6000 4750
@@
 $EndComp
 $Comp
-L VCC #PWR15
+L power:VCC #PWR15
 U 1 1 561C7507
 P 6000 4600
@@
 $EndComp
 $Comp
-L GND #PWR16
+L power:GND #PWR16
 U 1 1 561C7532
 P 6000 4900

Commit message: Update schematic components to latest library
Parts:
- C2: symbol device:C -> Device:C
Changed lines of the file:
@@
 EESchema Schematic File Version 4
-LIBS:mega-wifi-cache
-EELAYER 26 0
+EELAYER 30 0
 EELAYER END
 $Descr A4 11693 8268
@@
 	6700 4050 6750 4050
 $Comp
-L device:C C2
+L Device:C C2
 U 1 1 561C7483
 P 6000 4750

Commit message: Update to Rev.A2
Parts:
- C2: LCSC# (none) -> C2830722
- U2: LCSC# (none) -> C62389
Changed lines of the file:
@@
 Sheet 2 3
 Title "MegaWiFi"
-Date "2017-03-24"
-Rev "A1"
+Date "2021-10-31"
+Rev "A2"
 Comp "doragasu"
 Comment1 "License: CERN OHL 1.2"
@@
 F 3 "" H 6150 3350 60  0000 C CNN
 F 4 "S29GL032N90TFI030" H 6000 2850 60  0001 C CNN "manf#"
+F 5 "C62389" H 6000 2850 50  0001 C CNN "LCSC#"
 	1    6000 2850
 	1    0    0    -1
@@
 NoConn ~ 6700 3650
 $Comp
-L power:VCC #PWR14
+L power:VCC #PWR014
 U 1 1 561C7245
 P 6750 4050
-F 0 "#PWR14" H 6750 3900 50  0001 C CNN
+F 0 "#PWR014" H 6750 3900 50  0001 C CNN
 F 1 "VCC" H 6750 4200 50  0000 C CNN
 F 2 "" H 6750 4050 60  0000 C CNN
@@
 F 2 "Capacitors_SMD:C_0805" H 6038 4600 30  0001 C CNN
 F 3 "" H 6000 4750 60  0000 C CNN
+F 4 "C2830722" H 6000 4750 50  0001 C CNN "LCSC#"
 	1    6000 4750
 	1    0    0    -1
 $EndComp
 $Comp
-L power:VCC #PWR15
+L power:VCC #PWR015
 U 1 1 561C7507
 P 6000 4600
-F 0 "#PWR15" H 6000 4450 50  0001 C CNN
+F 0 "#PWR015" H 6000 4450 50  0001 C CNN
 F 1 "VCC" H 6000 4750 50  0000 C CNN
 F 2 "" H 6000 4600 60  0000 C CNN
@@
 $EndComp
 $Comp
-L power:GND #PWR16
+L power:GND #PWR016
 U 1 1 561C7532
 P 6000 4900
-F 0 "#PWR16" H 6000 4650 50  0001 C CNN
+F 0 "#PWR016" H 6000 4650 50  0001 C CNN
 F 1 "GND" H 6000 4750 50  0001 C CNN
 F 2 "" H 6000 4900 60  0000 C CNN
