File: wifi.sch (KiCad schematic (older format))
At the start: 19 parts, among them P1 CONN_01X02, Q1 2N7002, U1 SC16C550BIB48, U3 ESP-12E, Y1 NP

Commit message: Updated to latest KiCad and libraries version.
Parts:
- removed P1: CONN_01X02, Socket_Strips:Socket_Strip_Straight_1x02, symbol CONN_01X02
- added P1: Conn_01x02, Socket_Strips:Socket_Strip_Straight_1x02, symbol Connector:Conn_01x02
- C1, C3, C4, C5, C6: symbol C -> device:C
- D1: symbol LED -> device:LED
- Q1: symbol Q_NMOS_GSD -> device:Q_NMOS_GSD
- R1, R2, R3, R4, R5, R6, R7, R8: symbol R -> device:R
- U1: symbol SC16C550BIB48 -> doragasu:SC16C550BIB48
- U3: symbol ESP-12E -> ESP8266:ESP-12E
- Y1: symbol Crystal_Small -> device:Crystal_Small
Connections:
- net GND: now also P1.2 (Pin_2)
- net at U3.17 (GPIO2): now also P1.1 (Pin_1)
Changed lines of the file:
@@
-EESchema Schematic File Version 2
-LIBS:power
-LIBS:device
-LIBS:transistors
-LIBS:conn
-LIBS:linear
-LIBS:regul
-LIBS:74xx
-LIBS:cmos4000
-LIBS:adc-dac
-LIBS:memory
-LIBS:xilinx
-LIBS:microcontrollers
-LIBS:dsp
-LIBS:microchip
-LIBS:analog_switches
-LIBS:motorola
-LIBS:texas
-LIBS:intel
-LIBS:audio
-LIBS:interface
-LIBS:digital-audio
-LIBS:philips
-LIBS:display
-LIBS:cypress
-LIBS:siliconi
-LIBS:opto
-LIBS:atmel
-LIBS:contrib
-LIBS:valves
-LIBS:ESP8266
-LIBS:doragasu
+EESchema Schematic File Version 4
 LIBS:mega-wifi-cache
 EELAYER 26 0
@@
 $EndDescr
 $Comp
-L SC16C550BIB48 U1
+L doragasu:SC16C550BIB48 U1
 U 1 1 5619FAD2
 P 4950 3950
@@
 	9100 4600 9100 3650
 Wire Wire Line
-	9000 3650 9600 3650
+	9000 3650 9100 3650
 Wire Wire Line
 	5650 2550 9100 2550
@@
 	6250 4700 9200 4700
 Wire Wire Line
-	9200 4700 9200 3450
+	9200 4700 9200 3750
 Wire Wire Line
 	9200 3450 9000 3450
@@
 #W_RST
 $Comp
-L GND #PWR22
+L power:GND #PWR22
 U 1 1 5619FB0E
 P 9000 3750
@@
 	4250 3950 3950 3950
 $Comp
-L GND #PWR32
+L power:GND #PWR32
 U 1 1 561FA094
 P 4950 5550
@@
 $EndComp
 $Comp
-L VCC #PWR17
+L power:VCC #PWR17
 U 1 1 561FA1A0
 P 4950 2150
@@
 NoConn ~ 4250 5050
 $Comp
-L R R3
+L device:R R3
 U 1 1 5621824C
 P 3950 5100
@@
 	4250 5250 3950 5250
 $Comp
-L GND #PWR33
+L power:GND #PWR33
 U 1 1 562182B6
 P 3950 5650
@@
 $EndComp
 $Comp
-L VCC #PWR28
+L power:VCC #PWR28
 U 1 1 56218334
 P 3950 4950
@@
 $EndComp
 $Comp
-L Crystal_Small Y1
+L device:Crystal_Small Y1
 U 1 1 562186A7
 P 5800 5150
@@
 $EndComp
 $Comp
-L C C3
+L device:C C3
 U 1 1 562187DC
 P 6100 5050
@@
 $EndComp
 $Comp
-L C C4
+L device:C C4
 U 1 1 56218812
 P 6100 5250
@@
 $EndComp
 Wire Wire Line
-	5650 5050 5950 5050
+	5650 5050 5800 5050
 Connection ~ 5800 5050
 Wire Wire Line
-	5650 5250 5950 5250
+	5650 5250 5800 5250
 Connection ~ 5800 5250
 $Comp
-L GND #PWR30
+L power:GND #PWR30
 U 1 1 56218992
 P 6350 5300
@@
 	6250 5050 6350 5050
 Wire Wire Line
-	6350 5050 6350 5300
+	6350 5050 6350 5250
 Wire Wire Line
 	6250 5250 6350 5250
@@
 WARNING\n_________\n\nTo upload firmware on ESP8266 when pulling RESET high:\n- GPIO15 must be LOW.\n- GPIO0 must be LOW.\n- CH_PD must be HIGH.\n\nTo boot ESP8266 when pulling RESET high:\n- GPIO15 must be LOW.\n- GPIO0 must be HIGH.\n- CH_PD must be HIGH or the module will enter low power mode.
 $Comp
-L R R1
+L device:R R1
 U 1 1 5624E3A5
 P 3500 4550
@@
 $EndComp
 $Comp
-L R R2
+L device:R R2
 U 1 1 5624E420
 P 3750 4700
@@
 $EndComp
 Wire Wire Line
-	3650 4550 4250 4550
+	3650 4550 3750 4550
 Connection ~ 3750 4550
 Wire Wire Line
 	3350 4550 3200 4550
 $Comp
-L GND #PWR27
+L power:GND #PWR27
 U 1 1 5624E6E8
 P 3750 4850
@@
 $EndComp
 $Comp
-L GND #PWR25
+L power:GND #PWR25
 U 1 1 5624F0AE
 P 3600 4100
@@
 All CS pins must be active,\nbut only one IOR or IOW pin\nmust be active for operation.
 $Comp
-L C C1
+L device:C C1
 U 1 1 56250803
 P 4950 6150
@@
 $EndComp
 $Comp
-L C C6
+L device:C C6
 U 1 1 5625097E
 P 8050 5200
@@
 $EndComp
 $Comp
-L GND #PWR35
+L power:GND #PWR35
 U 1 1 56250A57
 P 4950 6300
@@
 $EndComp
 $Comp
-L GND #PWR31
+L power:GND #PWR31
 U 1 1 56250A89
 P 8050 5350
@@
 $EndComp
 $Comp
-L VCC #PWR34
+L power:VCC #PWR34
 U 1 1 56250ABB
 P 4950 6000
@@
 	3950 3350 4250 3350
 $Comp
-L ESP-12E U3
+L ESP8266:ESP-12E U3
 U 1 1 5619FAD9
 P 8100 3350
@@
 $EndComp
 Wire Wire Line
-	5650 2850 6900 2850
+	5650 2850 6550 2850
 Wire Wire Line
 	6550 2850 6550 3250
@@
 #W_PD
 $Comp
-L R R8
+L device:R R8
 U 1 1 56233843
 P 9800 3100
@@
 $EndComp
 Wire Wire Line
-	9000 3350 9350 3350
-$Comp
-L LED D1
+	9000 3350 9400 3350
+$Comp
+L device:LED D1
 U 1 1 562339B0
 P 9550 3350
+AR Path="/562339B0" Ref="D1"  Part="1"
+AR Path="/5619415C/562339B0" Ref="D1"  Part="1"
 F 0 "D1" H 9550 3550 50  0000 C CNN
 F 1 "LED" H 9550 3450 50  0000 C CNN
@@
 #W_DAT
 $Comp
-L R R7
+L device:R R7
 U 1 1 56237BB0
 P 9600 3900
@@
 Connection ~ 9100 3650
 $Comp
-L GND #PWR24
+L power:GND #PWR24
 U 1 1 56237CF0
 P 9600 4050
@@
 $EndComp
 $Comp
-L Q_NMOS_GSD Q1
+L device:Q_NMOS_GSD Q1
 U 1 1 56238C3B
 P 3850 5450
@@
 	4250 3850 3600 3850
 Wire Wire Line
-	3600 3850 3600 4100
+	3600 3850 3600 4050
 Connection ~ 3600 4050
 $Comp
-L R R6
+L device:R R6
 U 1 1 569B47C7
 P 9350 3900
@@
 $EndComp
 $Comp
-L GND #PWR23
+L power:GND #PWR23
 U 1 1 569B4859
 P 9350 4050
@@
 Connection ~ 9200 3750
 $Comp
-L R R5
+L device:R R5
 U 1 1 569B4F32
 P 7050 2850
@@
 NoConn ~ 7200 3150
 Wire Wire Line
-	9750 3350 9800 3350
+	9700 3350 9800 3350
 Wire Wire Line
 	9800 3350 9800 3250
@@
 	5650 3850 5650 3950
 $Comp
-L VCC #PWR29
+L power:VCC #PWR29
 U 1 1 56C051EB
 P 8050 5050
@@
 $EndComp
 $Comp
-L VCC #PWR19
+L power:VCC #PWR19
 U 1 1 56C0522C
 P 9800 2900
@@
 $EndComp
 $Comp
-L VCC #PWR18
+L power:VCC #PWR18
 U 1 1 56C05BB4
 P 7300 2850
@@
 $EndComp
 $Comp
-L VCC #PWR21
+L power:VCC #PWR21
 U 1 1 56C05E9A
 P 7200 3750
@@
 	0    -1   -1   0
 $EndComp
-$Comp
-L CONN_01X02 P1
-U 1 1 56C0650A
-P 10050 3600
-F 0 "P1" H 10128 3592 50  0000 L CNN
-F 1 "CONN_01X02" H 10127 3546 50  0001 L CNN
-F 2 "Socket_Strips:Socket_Strip_Straight_1x02" H 10050 3600 60  0001 C CNN
-F 3 "" H 10050 3600 60  0000 C CNN
-	1    10050 3600
-	1    0    0    -1
-$EndComp
 Wire Wire Line
 	9000 3550 9850 3550
 $Comp
-L GND #PWR20
+L power:GND #PWR20
 U 1 1 56C068A5
 P 9850 3650
@@
 VSYNC
 $Comp
-L C C5
+L device:C C5
 U 1 1 56C46DD0
 P 7050 4100
@@
 $EndComp
 $Comp
-L R R4
+L device:R R4
 U 1 1 56C46E52
 P 6850 3900
@@
 	6650 3900 6700 3900
 Wire Wire Line
-	7000 3900 7150 3900
+	7000 3900 7050 3900
 Wire Wire Line
 	7050 3950 7050 3900
 Connection ~ 7050 3900
 $Comp
-L GND #PWR26
+L power:GND #PWR26
 U 1 1 56C47761
 P 7050 4250
@@
 	1    0    0    -1
 $EndComp
+Wire Wire Line
+	5800 5050 5950 5050
+Wire Wire Line
+	5800 5250 5950 5250
+Wire Wire Line
+	6350 5250 6350 5300
+Wire Wire Line
+	3750 4550 4250 4550
+Wire Wire Line
+	9100 3650 9600 3650
+Wire Wire Line
+	3600 4050 3600 4100
+Wire Wire Line
+	9200 3750 9200 3450
+Wire Wire Line
+	6550 2850 6900 2850
+Wire Wire Line
+	7050 3900 7150 3900
+$Comp
+L Connector:Conn_01x02 P1
+U 1 1 5ACAF1FB
+P 10050 3550
+F 0 "P1" H 10129 3496 50  0000 L CNN
+F 1 "Conn_01x02" H 10130 3451 50  0001 L CNN
+F 2 "Socket_Strips:Socket_Strip_Straight_1x02" H 10050 3550 50  0001 C CNN
+F 3 "~" H 10050 3550 50  0001 C CNN
+	1    10050 3550
+	1    0    0    -1
+$EndComp

Commit message: Update schematic components to latest library
Parts:
- C1, C3, C4, C5, C6: symbol device:C -> Device:C
- D1: symbol device:LED -> Device:LED
- P1: symbol Connector:Conn_01x02 -> Connector_Generic:Conn_01x02
- Q1: symbol device:Q_NMOS_GSD -> Device:Q_NMOS_GSD
- R1, R2, R3, R4, R5, R6, R7, R8: symbol device:R -> Device:R
- Y1: symbol device:Crystal_Small -> Device:Crystal_Small
Changed lines of the file:
@@
 EESchema Schematic File Version 4
-LIBS:mega-wifi-cache
-EELAYER 26 0
+EELAYER 30 0
 EELAYER END
 $Descr A4 11693 8268
@@
 NoConn ~ 4250 5050
 $Comp
-L device:R R3
+L Device:R R3
 U 1 1 5621824C
 P 3950 5100
@@
 $EndComp
 $Comp
-L device:Crystal_Small Y1
+L Device:Crystal_Small Y1
 U 1 1 562186A7
 P 5800 5150
@@
 $EndComp
 $Comp
-L device:C C3
+L Device:C C3
 U 1 1 562187DC
 P 6100 5050
@@
 $EndComp
 $Comp
-L device:C C4
+L Device:C C4
 U 1 1 56218812
 P 6100 5250
@@
 WARNING\n_________\n\nTo upload firmware on ESP8266 when pulling RESET high:\n- GPIO15 must be LOW.\n- GPIO0 must be LOW.\n- CH_PD must be HIGH.\n\nTo boot ESP8266 when pulling RESET high:\n- GPIO15 must be LOW.\n- GPIO0 must be HIGH.\n- CH_PD must be HIGH or the module will enter low power mode.
 $Comp
-L device:R R1
+L Device:R R1
 U 1 1 5624E3A5
 P 3500 4550
@@
 $EndComp
 $Comp
-L device:R R2
+L Device:R R2
 U 1 1 5624E420
 P 3750 4700
@@
 All CS pins must be active,\nbut only one IOR or IOW pin\nmust be active for operation.
 $Comp
-L device:C C1
+L Device:C C1
 U 1 1 56250803
 P 4950 6150
@@
 $EndComp
 $Comp
-L device:C C6
+L Device:C C6
 U 1 1 5625097E
 P 8050 5200
@@
 #W_PD
 $Comp
-L device:R R8
+L Device:R R8
 U 1 1 56233843
 P 9800 3100
@@
 	9000 3350 9400 3350
 $Comp
-L device:LED D1
+L Device:LED D1
 U 1 1 562339B0
 P 9550 3350
@@
 #W_DAT
 $Comp
-L device:R R7
+L Device:R R7
 U 1 1 56237BB0
 P 9600 3900
@@
 $EndComp
 $Comp
-L device:Q_NMOS_GSD Q1
+L Device:Q_NMOS_GSD Q1
 U 1 1 56238C3B
 P 3850 5450
@@
 Connection ~ 3600 4050
 $Comp
-L device:R R6
+L Device:R R6
 U 1 1 569B47C7
 P 9350 3900
@@
 Connection ~ 9200 3750
 $Comp
-L device:R R5
+L Device:R R5
 U 1 1 569B4F32
 P 7050 2850
@@
 VSYNC
 $Comp
-L device:C C5
+L Device:C C5
 U 1 1 56C46DD0
 P 7050 4100
@@
 $EndComp
 $Comp
-L device:R R4
+L Device:R R4
 U 1 1 56C46E52
 P 6850 3900
@@
 	7050 3900 7150 3900
 $Comp
-L Connector:Conn_01x02 P1
+L Connector_Generic:Conn_01x02 P1
 U 1 1 5ACAF1FB
 P 10050 3550
+AR Path="/5ACAF1FB" Ref="P1"  Part="1"
+AR Path="/5619415C/5ACAF1FB" Ref="P1"  Part="1"
 F 0 "P1" H 10129 3496 50  0000 L CNN
 F 1 "Conn_01x02" H 10130 3451 50  0001 L CNN

Commit message: Update to Rev.A2
Parts:
- C1, C6: LCSC# (none) -> C2830722
- C3, C4: value NP -> 22p; LCSC# (none) -> C237185
- C5: value 100n -> NP; LCSC# (none) -> C2830722
- D1: value LED -> NP
- P1: value Conn_01x02 -> NP; footprint Socket_Strips:Socket_Strip_Straight_1x02 -> Connector_PinHeader_2.54mm:PinHeader_1x02_P2.54mm_Vertical
- Q1: LCSC# (none) -> C306856
- R1: LCSC# (none) -> C96345
- R3, R5, R6, R7: LCSC# (none) -> C2763777
- R4: value 1k -> NP
- R8: value 220 -> NP
- U1: LCSC# (none) -> C84320
- U3: LCSC# (none) -> C89297
- Y1: value NP -> 24 MHz; LCSC# (none) -> C259050
Other:
- note added: "ESP8266 boot options:\n_______________________\n\nTo upload firmware on ESP8266 when pulling RESET high:\n- GPIO15 must be LOW.\n- GPIO0 must be LOW.\n- CH_PD must be HIGH.\n\nTo boot ESP8266 when pulling RESET high:\n- GPIO15 must be LOW.\n- GPIO0 must be HIGH.\n- CH_PD must be HIGH or the module will enter low power mode."
- note removed: "WARNING\n_________\n\nTo upload firmware on ESP8266 when pulling RESET high:\n- GPIO15 must be LOW.\n- GPIO0 must be LOW.\n- CH_PD must be HIGH.\n\nTo boot ESP8266 when pulling RESET high:\n- GPIO15 must be LOW.\n- GPIO0 must be HIGH.\n- CH_PD must be HIGH or the module will enter low power mode."
Changed lines of the file:
@@
 Sheet 3 3
 Title "MegaWiFi"
-Date "2017-03-24"
-Rev "A1"
+Date "2021-10-31"
+Rev "A2"
 Comp "doragasu"
 Comment1 "License: CERN OHL 1.2"
@@
 F 3 "" H 4950 3950 60  0000 C CNN
 F 4 "SC16C550BIB48,151" H 4950 3950 60  0001 C CNN "manf#"
+F 5 "C84320" H 4950 3950 50  0001 C CNN "LCSC#"
 	1    4950 3950
 	1    0    0    -1
@@
 #W_RST
 $Comp
-L power:GND #PWR22
+L power:GND #PWR022
 U 1 1 5619FB0E
 P 9000 3750
-F 0 "#PWR22" H 9000 3500 50  0001 C CNN
+F 0 "#PWR022" H 9000 3500 50  0001 C CNN
 F 1 "GND" H 9000 3600 50  0001 C CNN
 F 2 "" H 9000 3750 60  0000 C CNN
@@
 	4250 3950 3950 3950
 $Comp
-L power:GND #PWR32
+L power:GND #PWR032
 U 1 1 561FA094
 P 4950 5550
-F 0 "#PWR32" H 4950 5300 50  0001 C CNN
+F 0 "#PWR032" H 4950 5300 50  0001 C CNN
 F 1 "GND" H 4950 5400 50  0001 C CNN
 F 2 "" H 4950 5550 60  0000 C CNN
@@
 $EndComp
 $Comp
-L power:VCC #PWR17
+L power:VCC #PWR017
 U 1 1 561FA1A0
 P 4950 2150
-F 0 "#PWR17" H 4950 2000 50  0001 C CNN
+F 0 "#PWR017" H 4950 2000 50  0001 C CNN
 F 1 "VCC" H 4950 2300 50  0000 C CNN
 F 2 "" H 4950 2150 60  0000 C CNN
@@
 F 2 "Resistors_SMD:R_0805" V 3880 5100 30  0001 C CNN
 F 3 "" H 3950 5100 30  0000 C CNN
+F 4 "C2763777" H 3950 5100 50  0001 C CNN "LCSC#"
 	1    3950 5100
 	1    0    0    -1
@@
 	4250 5250 3950 5250
 $Comp
-L power:GND #PWR33
+L power:GND #PWR033
 U 1 1 562182B6
 P 3950 5650
-F 0 "#PWR33" H 3950 5400 50  0001 C CNN
+F 0 "#PWR033" H 3950 5400 50  0001 C CNN
 F 1 "GND" H 3950 5500 50  0001 C CNN
 F 2 "" H 3950 5650 60  0000 C CNN
@@
 $EndComp
 $Comp
-L power:VCC #PWR28
+L power:VCC #PWR028
 U 1 1 56218334
 P 3950 4950
-F 0 "#PWR28" H 3950 4800 50  0001 C CNN
+F 0 "#PWR028" H 3950 4800 50  0001 C CNN
 F 1 "VCC" H 3950 5100 50  0000 C CNN
 F 2 "" H 3950 4950 60  0000 C CNN
@@
 P 5800 5150
 F 0 "Y1" V 5800 5300 50  0000 C CNN
-F 1 "NP" V 6000 5150 50  0000 C CNN
+F 1 "24 MHz" V 6000 5150 50  0000 C CNN
 F 2 "Crystals:Crystal_HC49-SD_SMD" H 5800 5150 60  0001 C CNN
 F 3 "" H 5800 5150 60  0000 C CNN
+F 4 "C259050" V 5800 5150 50  0001 C CNN "LCSC#"
 	1    5800 5150
 	0    1    1    0
@@
 P 6100 5050
 F 0 "C3" V 6050 5150 50  0000 L CNN
-F 1 "NP" V 6050 4900 50  0000 L CNN
+F 1 "22p" V 6050 5000 50  0000 R CNN
 F 2 "Capacitors_SMD:C_0805" H 6138 4900 30  0001 C CNN
 F 3 "" H 6100 5050 60  0000 C CNN
+F 4 "C237185" V 6100 5050 50  0001 C CNN "LCSC#"
 	1    6100 5050
 	0    1    1    0
@@
 P 6100 5250
 F 0 "C4" V 6050 5350 50  0000 L CNN
-F 1 "NP" V 6150 5100 50  0000 L CNN
+F 1 "22p" V 6150 5200 50  0000 R CNN
 F 2 "Capacitors_SMD:C_0805" H 6138 5100 30  0001 C CNN
 F 3 "" H 6100 5250 60  0000 C CNN
+F 4 "C237185" V 6100 5250 50  0001 C CNN "LCSC#"
 	1    6100 5250
 	0    1    1    0
@@
 Connection ~ 5800 5250
 $Comp
-L power:GND #PWR30
+L power:GND #PWR030
 U 1 1 56218992
 P 6350 5300
-F 0 "#PWR30" H 6350 5050 50  0001 C CNN
+F 0 "#PWR030" H 6350 5050 50  0001 C CNN
 F 1 "GND" H 6350 5150 50  0001 C CNN
 F 2 "" H 6350 5300 60  0000 C CNN
@@
 NoConn ~ 5650 3650
 Text Notes 650  7700 0    60   ~ 0
-WARNING\n_________\n\nTo upload firmware on ESP8266 when pulling RESET high:\n- GPIO15 must be LOW.\n- GPIO0 must be LOW.\n- CH_PD must be HIGH.\n\nTo boot ESP8266 when pulling RESET high:\n- GPIO15 must be LOW.\n- GPIO0 must be HIGH.\n- CH_PD must be HIGH or the module will enter low power mode.
+ESP8266 boot options:\n_______________________\n\nTo upload firmware on ESP8266 when pulling RESET high:\n- GPIO15 must be LOW.\n- GPIO0 must be LOW.\n- CH_PD must be HIGH.\n\nTo boot ESP8266 when pulling RESET high:\n- GPIO15 must be LOW.\n- GPIO0 must be HIGH.\n- CH_PD must be HIGH or the module will enter low power mode.
 $Comp
 L Device:R R1
@@
 F 2 "doragasu:JUMPER_0805" V 3430 4550 30  0001 C CNN
 F 3 "" H 3500 4550 30  0000 C CNN
+F 4 "C96345" H 3500 4550 50  0001 C CNN "LCSC#"
 	1    3500 4550
 	0    1    1    0
@@
 	3350 4550 3200 4550
 $Comp
-L power:GND #PWR27
+L power:GND #PWR027
 U 1 1 5624E6E8
 P 3750 4850
-F 0 "#PWR27" H 3750 4600 50  0001 C CNN
+F 0 "#PWR027" H 3750 4600 50  0001 C CNN
 F 1 "GND" H 3750 4700 50  0001 C CNN
 F 2 "" H 3750 4850 60  0000 C CNN
@@
 $EndComp
 $Comp
-L power:GND #PWR25
+L power:GND #PWR025
 U 1 1 5624F0AE
 P 3600 4100
-F 0 "#PWR25" H 3600 3850 50  0001 C CNN
+F 0 "#PWR025" H 3600 3850 50  0001 C CNN
 F 1 "GND" H 3600 3950 50  0001 C CNN
 F 2 "" H 3600 4100 60  0000 C CNN
@@
 F 2 "Capacitors_SMD:C_0805" H 4988 6000 30  0001 C CNN
 F 3 "" H 4950 6150 60  0000 C CNN
+F 4 "C2830722" H 4950 6150 50  0001 C CNN "LCSC#"
 	1    4950 6150
 	1    0    0    -1
@@
 F 2 "Capacitors_SMD:C_0805" H 8088 5050 30  0001 C CNN
 F 3 "" H 8050 5200 60  0000 C CNN
+F 4 "C2830722" H 8050 5200 50  0001 C CNN "LCSC#"
 	1    8050 5200
 	1    0    0    -1
 $EndComp
 $Comp
-L power:GND #PWR35
+L power:GND #PWR035
 U 1 1 56250A57
 P 4950 6300
-F 0 "#PWR35" H 4950 6050 50  0001 C CNN
+F 0 "#PWR035" H 4950 6050 50  0001 C CNN
 F 1 "GND" H 4950 6150 50  0001 C CNN
 F 2 "" H 4950 6300 60  0000 C CNN
@@
 $EndComp
 $Comp
-L power:GND #PWR31
+L power:GND #PWR031
 U 1 1 56250A89
 P 8050 5350
-F 0 "#PWR31" H 8050 5100 50  0001 C CNN
+F 0 "#PWR031" H 8050 5100 50  0001 C CNN
 F 1 "GND" H 8050 5200 50  0001 C CNN
 F 2 "" H 8050 5350 60  0000 C CNN
@@
 $EndComp
 $Comp
-L power:VCC #PWR34
+L power:VCC #PWR034
 U 1 1 56250ABB
 P 4950 6000
-F 0 "#PWR34" H 4950 5850 50  0001 C CNN
+F 0 "#PWR034" H 4950 5850 50  0001 C CNN
 F 1 "VCC" H 4950 6150 50  0000 C CNN
 F 2 "" H 4950 6000 60  0000 C CNN
@@
 F 3 "" H 8100 3350 50  0001 C CNN
 F 4 "1:$2" H 8100 3350 60  0001 C CNN "kicost:pricing"
+F 5 "C89297" H 8100 3350 50  0001 C CNN "LCSC#"
 	1    8100 3350
 	1    0    0    -1
@@
 P 9800 3100
 F 0 "R8" V 9700 3100 50  0000 C CNN
-F 1 "220" V 9800 3100 50  0000 C CNN
+F 1 "NP" V 9800 3100 50  0000 C CNN
 F 2 "Resistors_SMD:R_0805" V 9730 3100 30  0001 C CNN
 F 3 "" H 9800 3100 30  0000 C CNN
@@
 AR Path="/5619415C/562339B0" Ref="D1"  Part="1"
 F 0 "D1" H 9550 3550 50  0000 C CNN
-F 1 "LED" H 9550 3450 50  0000 C CNN
+F 1 "NP" H 9550 3450 50  0000 C CNN
 F 2 "LEDs:LED-0603" H 9550 3350 60  0001 C CNN
 F 3 "" H 9550 3350 60  0000 C CNN
@@
 F 2 "Resistors_SMD:R_0805" V 9530 3900 30  0001 C CNN
 F 3 "" H 9600 3900 30  0000 C CNN
+F 4 "C2763777" H 9600 3900 50  0001 C CNN "LCSC#"
 	1    9600 3900
 	-1   0    0    1
@@
 Connection ~ 9100 3650
 $Comp
-L power:GND #PWR24
+L power:GND #PWR024
 U 1 1 56237CF0
 P 9600 4050
-F 0 "#PWR24" H 9600 3800 50  0001 C CNN
+F 0 "#PWR024" H 9600 3800 50  0001 C CNN
 F 1 "GND" H 9600 3900 50  0001 C CNN
 F 2 "" H 9600 4050 60  0000 C CNN
@@
 F 3 "" H 3850 5450 60  0000 C CNN
 F 4 "2N7002E" H 3850 5450 60  0001 C CNN "manf#"
+F 5 "C306856" H 3850 5450 50  0001 C CNN "LCSC#"
 	1    3850 5450
 	1    0    0    -1
@@
 F 2 "Resistors_SMD:R_0805" V 9280 3900 30  0001 C CNN
 F 3 "" H 9350 3900 30  0000 C CNN
+F 4 "C2763777" H 9350 3900 50  0001 C CNN "LCSC#"
 	1    9350 3900
 	-1   0    0    1
 $EndComp
 $Comp
-L power:GND #PWR23
+L power:GND #PWR023
 U 1 1 569B4859
 P 9350 4050
-F 0 "#PWR23" H 9350 3800 50  0001 C CNN
+F 0 "#PWR023" H 9350 3800 50  0001 C CNN
 F 1 "GND" H 9350 3900 50  0001 C CNN
 F 2 "" H 9350 4050 60  0000 C CNN
@@
 F 2 "Resistors_SMD:R_0805" V 6980 2850 30  0001 C CNN
 F 3 "" H 7050 2850 30  0000 C CNN
+F 4 "C2763777" H 7050 2850 50  0001 C CNN "LCSC#"
 	1    7050 2850
 	0    -1   -1   0
@@
 	5650 3850 5650 3950
 $Comp
-L power:VCC #PWR29
+L power:VCC #PWR029
 U 1 1 56C051EB
 P 8050 5050
-F 0 "#PWR29" H 8050 4900 50  0001 C CNN
+F 0 "#PWR029" H 8050 4900 50  0001 C CNN
 F 1 "VCC" H 8050 5200 50  0000 C CNN
 F 2 "" H 8050 5050 60  0000 C CNN
@@
 $EndComp
 $Comp
-L power:VCC #PWR19
+L power:VCC #PWR019
 U 1 1 56C0522C
 P 9800 2900
-F 0 "#PWR19" H 9800 2750 50  0001 C CNN
+F 0 "#PWR019" H 9800 2750 50  0001 C CNN
 F 1 "VCC" H 9800 3050 50  0000 C CNN
 F 2 "" H 9800 2900 60  0000 C CNN
@@
 $EndComp
 $Comp
-L power:VCC #PWR18
+L power:VCC #PWR018
 U 1 1 56C05BB4
 P 7300 2850
-F 0 "#PWR18" H 7300 2700 50  0001 C CNN
+F 0 "#PWR018" H 7300 2700 50  0001 C CNN
 F 1 "VCC" H 7300 3000 50  0000 C CNN
 F 2 "" H 7300 2850 60  0000 C CNN
@@
 $EndComp
 $Comp
-L power:VCC #PWR21
+L power:VCC #PWR021
 U 1 1 56C05E9A
 P 7200 3750
-F 0 "#PWR21" H 7200 3600 50  0001 C CNN
+F 0 "#PWR021" H 7200 3600 50  0001 C CNN
 F 1 "VCC" V 7200 3950 50  0000 C CNN
 F 2 "" H 7200 3750 60  0000 C CNN
@@
 	9000 3550 9850 3550
 $Comp
-L power:GND #PWR20
+L power:GND #PWR020
 U 1 1 56C068A5
 P 9850 3650
-F 0 "#PWR20" H 9850 3400 50  0001 C CNN
+F 0 "#PWR020" H 9850 3400 50  0001 C CNN
 F 1 "GND" H 9850 3500 50  0001 C CNN
 F 2 "" H 9850 3650 60  0000 C CNN
@@
 P 7050 4100
 F 0 "C5" H 7075 4200 50  0000 L CNN
-F 1 "100n" H 7075 4000 50  0000 L CNN
+F 1 "NP" H 7075 4000 50  0000 L CNN
 F 2 "Capacitors_SMD:C_0805" H 7088 3950 30  0001 C CNN
 F 3 "" H 7050 4100 60  0000 C CNN
+F 4 "C2830722" H 7050 4100 50  0001 C CNN "LCSC#"
 	1    7050 4100
 	-1   0    0    -1
@@
 P 6850 3900
 F 0 "R4" V 6950 3950 50  0000 R CNN
-F 1 "1k" V 6850 3950 50  0000 R CNN
+F 1 "NP" V 6850 3950 50  0000 R CNN
 F 2 "Resistors_SMD:R_0805" V 6780 3900 30  0001 C CNN
 F 3 "" H 6850 3900 30  0000 C CNN
@@
 $EndComp
 Wire Wire Line
-	7200 3350 6650 3350
-Wire Wire Line
 	6650 3350 6650 3900
 Wire Wire Line
@@
 Connection ~ 7050 3900
 $Comp
-L power:GND #PWR26
+L power:GND #PWR026
 U 1 1 56C47761
 P 7050 4250
-F 0 "#PWR26" H 7050 4000 50  0001 C CNN
+F 0 "#PWR026" H 7050 4000 50  0001 C CNN
 F 1 "GND" H 7050 4100 50  0001 C CNN
 F 2 "" H 7050 4250 60  0000 C CNN
@@
 AR Path="/5ACAF1FB" Ref="P1"  Part="1"
 AR Path="/5619415C/5ACAF1FB" Ref="P1"  Part="1"
-F 0 "P1" H 10129 3496 50  0000 L CNN
-F 1 "Conn_01x02" H 10130 3451 50  0001 L CNN
-F 2 "Socket_Strips:Socket_Strip_Straight_1x02" H 10050 3550 50  0001 C CNN
+F 0 "P1" H 10150 3550 50  0000 L CNN
+F 1 "NP" H 10150 3450 50  0000 L CNN
+F 2 "Connector_PinHeader_2.54mm:PinHeader_1x02_P2.54mm_Vertical" H 10050 3550 50  0001 C CNN
 F 3 "~" H 10050 3550 50  0001 C CNN
 	1    10050 3550
 	1    0    0    -1
 $EndComp
+Wire Wire Line
+	7200 3350 6650 3350
 $EndSCHEMATC
